Commit message: fix: end effector flange joint coordinates are now in the correct location

File: urdf/mecabot.urdf.xacro (robot description, xacro)
@@ -92,5 +92,5 @@
 	<link name="end_effector_flange">
 		<visual>
-			<origin rpy="${pi/2} 0 0" xyz="0 0 0"/>
+			<origin rpy="${pi/2} 0 0" xyz="0 0 -0.1644"/>
 			<geometry>
 				<mesh filename="package://robotic_arm_model/mesh/link_6.stl" scale="0.01 0.01 0.01"/>
@@ -101,5 +101,6 @@
 		<parent link="link_5" />
 		<child link="end_effector_flange" />
-		<origin rpy="0 0 0" xyz="0 0 -0.89475" />
+		<!-- 89475 -->
+		<origin rpy="0 0 0" xyz="0 0 -0.73035" />
 		<axis xyz="0 0 1"/>
 		<limit lower="-${pi/2}" upper="${pi/2}" effort="30" velocity="10" />

Commit message: chore: gazebo launch file

File: urdf/mecabot.urdf.xacro (robot description, xacro)
@@ -1,4 +1,30 @@
 <?xml version="1.0" encoding="UTF-8"?>
 <robot xmlns:xacro="http://www.ros.org/wiki/xacro" name="block-robotics">
+	<xacro:macro name="defaultInertial" params="mass">
+		<inertial>
+			<mass value="${mass}"/>
+			<inertia ixx="1" ixy="0" ixz="0" iyy="1" iyz="0" izz="1"/>
+		</inertial>
+	</xacro:macro>
+	<xacro:macro name="defaultTransmission" params="number">
+		<transmission name="transmission_${number}">
+			<type>
+				transmission_interface/SimpleTransmission
+			</type>
+			<joint name="joint_${number}">
+				<hardwareInterface>
+					hardware_interface/PositionJointInterface
+				</hardwareInterface>
+			</joint>
+			<actuator name="motor_${number}">
+				<hardwareInterface>
+					hardware_interface/PositionJointInterface
+				</hardwareInterface>
+				<mechanicalReduction>
+					1
+				</mechanicalReduction>
+			</actuator>
+		</transmission>
+	</xacro:macro>
 	<link name="world" />
 	<link name="base_link">
@@ -9,4 +35,11 @@
 			</geometry>
 		</visual>
+		<collision>
+			<origin rpy="${pi/2} 0 0" xyz="0 0 0"/>
+			<geometry>
+				<mesh filename="package://robotic_arm_model/mesh/base_link.stl" scale="0.01 0.01 0.01"/>
+			</geometry>
+		</collision>
+		<xacro:defaultInertial mass="1.0"/>
 	</link>
 	<joint name="virtual_joint" type="fixed">
@@ -16,4 +49,5 @@
 	</joint>
 	<link name="link_1">
+		<xacro:defaultInertial mass="0.25"/>
 		<visual>
 			<origin rpy="${pi/2} 0 0" xyz="0 0 0.5"/>
@@ -22,4 +56,10 @@
 			</geometry>
 		</visual>
+		<collision>
+			<origin rpy="${pi/2} 0 0" xyz="0 0 0.5"/>
+			<geometry>
+				<mesh filename="package://robotic_arm_model/mesh/link_1.stl" scale="0.01 0.01 0.01"/>
+			</geometry>
+		</collision>
 	</link>
 	<joint name="joint_1" type="revolute">
@@ -31,4 +71,5 @@
 	</joint>
 	<link name="link_2">
+		<xacro:defaultInertial mass="0.3"/>
 		<visual>
 			<origin rpy="${pi/2} 0 0" xyz="0 -0.21078 -0.28624"/>
@@ -37,4 +78,10 @@
 			</geometry>
 		</visual>
+		<collision>
+			<origin rpy="${pi/2} 0 0" xyz="0 -0.21078 -0.28624"/>
+			<geometry>
+				<mesh filename="package://robotic_arm_model/mesh/link_2.stl" scale="0.01 0.01 0.01"/>
+			</geometry>
+		</collision>
 	</link>
 	<joint name="joint_2" type="revolute">
@@ -46,4 +93,5 @@
 	</joint>
 	<link name="link_3">
+		<xacro:defaultInertial mass="0.3"/>
 		<visual>
 			<origin rpy="${pi/2} 0 0" xyz="0.03556 0 0"/>
@@ -52,4 +100,10 @@
 			</geometry>
 		</visual>
+		<collision>
+			<origin rpy="${pi/2} 0 0" xyz="0.03556 0 0"/>
+			<geometry>
+				<mesh filename="package://robotic_arm_model/mesh/link_3.stl" scale="0.01 0.01 0.01"/>
+			</geometry>
+		</collision>
 	</link>
 	<joint name="joint_3" type="revolute">
@@ -61,4 +115,5 @@
 	</joint>
 	<link name="link_4">
+		<xacro:defaultInertial mass="0.25"/>
 		<visual>
 			<origin rpy="0 0 0" xyz="-0.2225 -0.35266 0.057835"/>
@@ -67,4 +122,10 @@
 			</geometry>
 		</visual>
+		<collision>
+			<origin rpy="0 0 0" xyz="-0.2225 -0.35266 0.057835"/>
+			<geometry>
+				<mesh filename="package://robotic_arm_model/mesh/link_4.stl" scale="0.01 0.01 0.01"/>
+			</geometry>
+		</collision>
 	</link>
 	<joint name="joint_4" type="revolute">
@@ -76,4 +137,5 @@
 	</joint>
 	<link name="link_5">
+		<xacro:defaultInertial mass="0.2"/>
 		<visual>
 			<origin rpy="0 ${pi} 0" xyz="0.0885 -0.32762 -0.5529"/>
@@ -82,4 +144,10 @@
 			</geometry>
 		</visual>
+		<collision>
+			<origin rpy="0 ${pi} 0" xyz="0.0885 -0.32762 -0.5529"/>
+			<geometry>
+				<mesh filename="package://robotic_arm_model/mesh/link_5.stl" scale="0.01 0.01 0.01"/>
+			</geometry>
+		</collision>
 	</link>
 	<joint name="joint_5" type="revolute">
@@ -91,4 +159,5 @@
 	</joint>
 	<link name="end_effector_flange">
+		<xacro:defaultInertial mass="0.01"/>
 		<visual>
 			<origin rpy="${pi/2} 0 0" xyz="0 0 -0.1644"/>
@@ -97,4 +166,10 @@
 			</geometry>
 		</visual>
+		<collision>
+			<origin rpy="${pi/2} 0 0" xyz="0 0 -0.1644"/>
+			<geometry>
+				<mesh filename="package://robotic_arm_model/mesh/link_6.stl" scale="0.01 0.01 0.01"/>
+			</geometry>
+		</collision>
 	</link>
 	<joint name="joint_6" type="revolute">
@@ -106,3 +181,16 @@
 		<limit lower="-${pi/2}" upper="${pi/2}" effort="30" velocity="10" />
 	</joint>
+	<xacro:defaultTransmission number="1"/>
+	<xacro:defaultTransmission number="2"/>
+	<xacro:defaultTransmission number="3"/>
+	<xacro:defaultTransmission number="4"/>
+	<xacro:defaultTransmission number="5"/>
+	<xacro:defaultTransmission number="6"/>
+	<gazebo>
+		<plugin name="gazebo_ros_control" filename="libgazebo_ros_control.so">s
+			<robotNamespace>/mecabot</robotNamespace>
+			<robotSimType>gazebo_ros_control/DefaultRobotHWSim</robotSimType>
+			<legacyModeNS>true</legacyModeNS>
+		</plugin>
+	</gazebo>
 </robot>

Commit message: chore: gazebo simulation

File: urdf/mecabot.urdf.xacro (robot description, xacro)
@@ -51,5 +51,5 @@
 		<xacro:defaultInertial mass="0.25"/>
 		<visual>
-			<origin rpy="${pi/2} 0 0" xyz="0 0 0.5"/>
+			<origin rpy="${pi/2} 0 0" xyz="0 0 0"/>
 			<geometry>
 				<mesh filename="package://robotic_arm_model/mesh/link_1.stl" scale="0.01 0.01 0.01"/>
@@ -57,5 +57,5 @@
 		</visual>
 		<collision>
-			<origin rpy="${pi/2} 0 0" xyz="0 0 0.5"/>
+			<origin rpy="${pi/2} 0 0" xyz="0 0 0"/>
 			<geometry>
 				<mesh filename="package://robotic_arm_model/mesh/link_1.stl" scale="0.01 0.01 0.01"/>
@@ -66,5 +66,5 @@
 		<parent link="base_link" />
 		<child link="link_1" />
-		<origin rpy="0 0 0" xyz="0 0 0" />
+		<origin rpy="0 0 0" xyz="0 0 0.5" />
 		<axis xyz="0 0 1"/>
 		<limit lower="-${pi/2}" upper="${pi/2}" effort="30" velocity="10" />
@@ -88,5 +88,5 @@
 		<parent link="link_1" />
 		<child link="link_2" />
-		<origin rpy="0 0 0" xyz="0 0 0.95" />
+		<origin rpy="0 0 0" xyz="0 0 0.45" />
 		<axis xyz="1 0 0"/>
 		<limit lower="-${pi/2}" upper="${pi/2}" effort="30" velocity="10" />
